File: 8x8x8 cube/baseboard.sch (EAGLE design)
At the start: 100 parts, among them IC1 LM321MF, J1 CONNECTOR-HEADER-2X2P2X2P-2.5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, J10 CONNECTOR-HEADER-2X2P2X2P-2.5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, J11 CONNECTOR-HEADER-2X2P2X2P-2.5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, J12 CONNECTOR-HEADER-2X2P2X2P-2.5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, J13 CONNECTOR-HEADER-2X2P2X2P-2.5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, J14 CONNECTOR-HEADER-2X2P2X2P-2.5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, J15 CONNECTOR-HEADER-2X2P2X2P-2.5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, J16 CONNECTOR-HEADER-2X2P2X2P-2.5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, J17 CONNECTOR-HEADER-2X2P2X2P-2.5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, J18 CONNECTOR-HEADER-2X2P2X2P-2.5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, J19 CONNECTOR-HEADER-2X2P2X2P-2.5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, J2 CONNECTOR-HEADER-2X2P2X2P-2.5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, J20 CONNECTOR-HEADER-2X2P2X2P-2.5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, J21 CONNECTOR-HEADER-2X2P2X2P-2.5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, J22 CONNECTOR-HEADER-2X2P2X2P-2.5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, J23 CONNECTOR-HEADER-2X2P2X2P-2.5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, J24 CONNECTOR-HEADER-2X2P2X2P-2.5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, J25 CONNECTOR-HEADER-2X2P2X2P-2.5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, J26 CONNECTOR-HEADER-2X2P2X2P-2.5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, J27 CONNECTOR-HEADER-2X2P2X2P-2.5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, J28 CONNECTOR-HEADER-2X2P2X2P-2.5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, J29 CONNECTOR-HEADER-2X2P2X2P-2.5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, J3 CONNECTOR-HEADER-2X2P2X2P-2.5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, J30 CONNECTOR-HEADER-2X2P2X2P-2.5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, J31 CONNECTOR-HEADER-2X2P2X2P-2.5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, J32 CONNECTOR-HEADER-2X2P2X2P-2.5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, J33 CONNECTOR-HEADER-2X2P2X2P-2.5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, J34 CONNECTOR-HEADER-2X2P2X2P-2.5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, J35 CONNECTOR-HEADER-2X2P2X2P-2.5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, J36 CONNECTOR-HEADER-2X2P2X2P-2.5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, J37 CONNECTOR-HEADER-2X2P2X2P-2.5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, J38 CONNECTOR-HEADER-2X2P2X2P-2.5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, J39 CONNECTOR-HEADER-2X2P2X2P-2.5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, J4 CONNECTOR-HEADER-2X2P2X2P-2.5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, J40 CONNECTOR-HEADER-2X2P2X2P-2.5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, J41 CONNECTOR-HEADER-2X2P2X2P-2.5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, J42 CONNECTOR-HEADER-2X2P2X2P-2.5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, J43 CONNECTOR-HEADER-2X2P2X2P-2.5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, J44 CONNECTOR-HEADER-2X2P2X2P-2.5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, J45 CONNECTOR-HEADER-2X2P2X2P-2.5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, J46 CONNECTOR-HEADER-2X2P2X2P-2.5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, J47 CONNECTOR-HEADER-2X2P2X2P-2.5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, J48 CONNECTOR-HEADER-2X2P2X2P-2.5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, J49 CONNECTOR-HEADER-2X2P2X2P-2.5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, J5 CONNECTOR-HEADER-2X2P2X2P-2.5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, J50 CONNECTOR-HEADER-2X2P2X2P-2.5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, J51 CONNECTOR-HEADER-2X2P2X2P-2.5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, J52 CONNECTOR-HEADER-2X2P2X2P-2.5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, J53 CONNECTOR-HEADER-2X2P2X2P-2.5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, J54 CONNECTOR-HEADER-2X2P2X2P-2.5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, J55 CONNECTOR-HEADER-2X2P2X2P-2.5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, J56 CONNECTOR-HEADER-2X2P2X2P-2.5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, J57 CONNECTOR-HEADER-2X2P2X2P-2.5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, J58 CONNECTOR-HEADER-2X2P2X2P-2.5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, J59 CONNECTOR-HEADER-2X2P2X2P-2.5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, J6 CONNECTOR-HEADER-2X2P2X2P-2.5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, J60 CONNECTOR-HEADER-2X2P2X2P-2.5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, J61 CONNECTOR-HEADER-2X2P2X2P-2.5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, J62 CONNECTOR-HEADER-2X2P2X2P-2.5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, J63 CONNECTOR-HEADER-2X2P2X2P-2.5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, J64 CONNECTOR-HEADER-2X2P2X2P-2.5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, J7 CONNECTOR-HEADER-2X2P2X2P-2.5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, J8 CONNECTOR-HEADER-2X2P2X2P-2.5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, J9 CONNECTOR-HEADER-2X2P2X2P-2.5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, Q3 MOSFET-N-044020001, U2 ADXL335

Commit message: updated to rev 7
Parts:
- removed IC1: LM321MF, linear:LM321MF
- added BUTTON: BUTTON-4P4P-12X12X6H, OPL Eagle Library:BUTTON-4P4P-12X12X6H
- added GOLD_ORB_SM1: OSHWLOGO_GOLD_ORB_MED, NBitWonder:OSHWLOGO_GOLD_ORB_MED
- added M1: MICROPHONE, OPL Eagle Library:MICROPHONE
- added Q4: SS8550, OPL Eagle Library:TRANSISTOR-PNP-041003001
- added R14, R15, R16: 10K, OPL Eagle Library:R-0603
- added R17: 100K, OPL Eagle Library:R-0603
- C1, C2: device OPL Eagle Library:C-POLARCAPACITOR-E5-8.5 -> OPL Eagle Library:C-POLAR
- C4: value 100pF -> DNP
- Q1, Q3: value MOSFET-N-044020001 -> 2N7002
- Q2: value FDD4141TO252 -> FDD6637
- R1, R6: value (none) -> 10K
- R13: value 100K -> 4.7K
- R7: value 2M -> DNP
- SV1: device con-amp-mt:S04P -> OPL Eagle Library:CON-S04P
- U$1: value MICROPHONE -> L3D-LOGOL3DCUBE-LOGO-0.8X2.5; device OPL Eagle Library:MICROPHONE -> OPL Eagle Library:L3D-LOGOL3DCUBE-LOGO-0.8X2.5
- U1: value (none) -> ADXL335; device OPL Eagle Library:TRANSISTOR-PNP-041003001 -> OPL Eagle Library:ADXL335
- U2: value ADXL335 -> LM321MF; device OPL Eagle Library:ADXL335 -> linear:LM321MF
- renumbered 2N7002 to Q1, FDD6637 to Q2
Connections:
- removed net D3: JP2.9
- new net MODE: BUTTON.A0, BUTTON.A1, JP2.9, R16.2
- new net N$71: JP1.6, R14.2, R15.1
- net +3V3: now also R16.1, R6.1, U1.VSS1, U1.VSS2, U2.V+; no longer IC1.V+, U2.VSS1, U2.VSS2
- net +5V: now also Q4.E; no longer R6.1, SV1-1.S, U1.E
- net GND: now also BUTTON.B0, BUTTON.B1, M1.GND, R15.2, U1.COM1, U1.COM2, U1.COM3, U1.COM4, U2.V-; no longer IC1.V-, U$1.GND, U2.COM1, U2.COM2, U2.COM3, U2.COM4
- net N$32: now also U2.OUT; no longer IC1.OUT
- net N$65: now also Q4.B; no longer U1.B
- net N$66: now also R17.1, U2.-IN; no longer IC1.-IN
- net N$67: now also Q4.C; no longer U1.C
- net N$69: now also R17.2, U2.+IN; no longer IC1.+IN
- net N$72: now also M1.IN; no longer U$1.IN
- net V+: now also R14.1, SV1-1.S; no longer JP1.6
- net XOUT: now also U1.X; no longer U2.X
- net YOUT: now also U1.Y; no longer U2.Y
- net ZOUT: now also U1.Z; no longer U2.Z
Other:
- moved on the sheet: R8
