File: 8x8x8 cube/Base Board.brd (EAGLE design)
At the start: 170 x 170 mm, 132 parts, among them J1 CONNECTOR-HEADER-2X2P2X2P-2.5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, J10 CONNECTOR-HEADER-2X2P2X2P-2.5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, J11 CONNECTOR-HEADER-2X2P2X2P-2.5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, J12 CONNECTOR-HEADER-2X2P2X2P-2.5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, J13 CONNECTOR-HEADER-2X2P2X2P-2.5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, J14 CONNECTOR-HEADER-2X2P2X2P-2.5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, J15 CONNECTOR-HEADER-2X2P2X2P-2.5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, J16 CONNECTOR-HEADER-2X2P2X2P-2.5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, J17 CONNECTOR-HEADER-2X2P2X2P-2.5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, J18 CONNECTOR-HEADER-2X2P2X2P-2.5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, J19 CONNECTOR-HEADER-2X2P2X2P-2.5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, J2 CONNECTOR-HEADER-2X2P2X2P-2.5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, J20 CONNECTOR-HEADER-2X2P2X2P-2.5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, J21 CONNECTOR-HEADER-2X2P2X2P-2.5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, J22 CONNECTOR-HEADER-2X2P2X2P-2.5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, J23 CONNECTOR-HEADER-2X2P2X2P-2.5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, J24 CONNECTOR-HEADER-2X2P2X2P-2.5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, J25 CONNECTOR-HEADER-2X2P2X2P-2.5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, J26 CONNECTOR-HEADER-2X2P2X2P-2.5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, J27 CONNECTOR-HEADER-2X2P2X2P-2.5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, J28 CONNECTOR-HEADER-2X2P2X2P-2.5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, J29 CONNECTOR-HEADER-2X2P2X2P-2.5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, J3 CONNECTOR-HEADER-2X2P2X2P-2.5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, J30 CONNECTOR-HEADER-2X2P2X2P-2.5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, J31 CONNECTOR-HEADER-2X2P2X2P-2.5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, J32 CONNECTOR-HEADER-2X2P2X2P-2.5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, J33 CONNECTOR-HEADER-2X2P2X2P-2.5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, J34 CONNECTOR-HEADER-2X2P2X2P-2.5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, J35 CONNECTOR-HEADER-2X2P2X2P-2.5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, J36 CONNECTOR-HEADER-2X2P2X2P-2.5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, J37 CONNECTOR-HEADER-2X2P2X2P-2.5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, J38 CONNECTOR-HEADER-2X2P2X2P-2.5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, J39 CONNECTOR-HEADER-2X2P2X2P-2.5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, J4 CONNECTOR-HEADER-2X2P2X2P-2.5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, J40 CONNECTOR-HEADER-2X2P2X2P-2.5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, J41 CONNECTOR-HEADER-2X2P2X2P-2.5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, J42 CONNECTOR-HEADER-2X2P2X2P-2.5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, J43 CONNECTOR-HEADER-2X2P2X2P-2.5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, J44 CONNECTOR-HEADER-2X2P2X2P-2.5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, J45 CONNECTOR-HEADER-2X2P2X2P-2.5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, J46 CONNECTOR-HEADER-2X2P2X2P-2.5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, J47 CONNECTOR-HEADER-2X2P2X2P-2.5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, J48 CONNECTOR-HEADER-2X2P2X2P-2.5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, J49 CONNECTOR-HEADER-2X2P2X2P-2.5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, J5 CONNECTOR-HEADER-2X2P2X2P-2.5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, J50 CONNECTOR-HEADER-2X2P2X2P-2.5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, J51 CONNECTOR-HEADER-2X2P2X2P-2.5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, J52 CONNECTOR-HEADER-2X2P2X2P-2.5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, J53 CONNECTOR-HEADER-2X2P2X2P-2.5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, J54 CONNECTOR-HEADER-2X2P2X2P-2.5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, J55 CONNECTOR-HEADER-2X2P2X2P-2.5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, J56 CONNECTOR-HEADER-2X2P2X2P-2.5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, J57 CONNECTOR-HEADER-2X2P2X2P-2.5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, J58 CONNECTOR-HEADER-2X2P2X2P-2.5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, J59 CONNECTOR-HEADER-2X2P2X2P-2.5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, J6 CONNECTOR-HEADER-2X2P2X2P-2.5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, J60 CONNECTOR-HEADER-2X2P2X2P-2.5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, J61 CONNECTOR-HEADER-2X2P2X2P-2.5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, J62 CONNECTOR-HEADER-2X2P2X2P-2.5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, J63 CONNECTOR-HEADER-2X2P2X2P-2.5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, J64 CONNECTOR-HEADER-2X2P2X2P-2.5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, J65 CONNECTOR-HEADER-8P-3460290P1, J66 CONNECTOR-HEADER-8P-3460290P1, J67 CONNECTOR-HEADER-8P-3460290P1, J68 CONNECTOR-HEADER-6P-3460270P1, J7 CONNECTOR-HEADER-2X2P2X2P-2.5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, J8 CONNECTOR-HEADER-2X2P2X2P-2.5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, J9 CONNECTOR-HEADER-2X2P2X2P-2.5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, M1 MICROPHONE, Q1 2N7002, Q2 FDD6637, Q3 2N7002, Q4 SS8550, U1 ADXL335, U3 LMV324IDR-1100030P1

Commit message: updated 8x bom, schematic and layout for the baseboard
Parts:
- R13: value 4.3K -> 4.7K
Connections:
- net JOIN_WIFI renamed MODE
- net ONLINE-OFFLINE renamed SWITCH
Changed lines of the file:
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@@
 <?xml version="1.0" encoding="utf-8"?>
 <!DOCTYPE eagle SYSTEM "eagle.dtd">
-<eagle version="7.1.0">
+<eagle version="7.2.0">
 <drawing>
 <settings>
@@
 <grid distance="1" unitdist="mil" unit="mil" style="lines" multiple="1" display="yes" altdistance="0.025" altunitdist="inch" altunit="inch"/>
 <layers>
-<layer number="1" name="Top" color="12" fill="1" visible="yes" active="yes"/>
+<layer number="1" name="Top" color="12" fill="1" visible="no" active="yes"/>
 <layer number="2" name="Route2" color="1" fill="3" visible="no" active="no"/>
 <layer number="3" name="Route3" color="4" fill="3" visible="no" active="no"/>
@@
 <layer number="14" name="Route14" color="1" fill="6" visible="no" active="no"/>
 <layer number="15" name="Route15" color="4" fill="6" visible="no" active="no"/>
-<layer number="16" name="Bottom" color="9" fill="1" visible="yes" active="yes"/>
-<layer number="17" name="Pads" color="3" fill="1" visible="yes" active="yes"/>
-<layer number="18" name="Vias" color="2" fill="1" visible="yes" active="yes"/>
-<layer number="19" name="Unrouted" color="10" fill="1" visible="yes" active="yes"/>
+<layer number="16" name="Bottom" color="9" fill="1" visible="no" active="yes"/>
+<layer number="17" name="Pads" color="3" fill="1" visible="no" active="yes"/>
+<layer number="18" name="Vias" color="2" fill="1" visible="no" active="yes"/>
+<layer number="19" name="Unrouted" color="10" fill="1" visible="no" active="yes"/>
 <layer number="20" name="Dimension" color="7" fill="1" visible="yes" active="yes"/>
 <layer number="21" name="tPlace" color="5" fill="1" visible="yes" active="yes"/>
@@
 <layer number="25" name="tNames" color="6" fill="1" visible="yes" active="yes"/>
 <layer number="26" name="bNames" color="6" fill="1" visible="no" active="yes"/>
-<layer number="27" name="tValues" color="7" fill="1" visible="no" active="yes"/>
+<layer number="27" name="tValues" color="7" fill="1" visible="yes" active="yes"/>
 <layer number="28" name="bValues" color="7" fill="1" visible="no" active="yes"/>
 <layer number="29" name="tStop" color="7" fill="3" visible="no" active="yes"/>
@@
 <attribute name="VALUE" x="112.0347" y="129.8538" size="0.6096" layer="27" ratio="10" rot="R270"/>
 </element>
-<element name="R13" library="OPL Eagle Library" package="R0603" value="4.3K" x="148.2634" y="126.7804" smashed="yes" rot="R270">
+<element name="R13" library="OPL Eagle Library" package="R0603" value="4.7K" x="148.2634" y="126.7804" smashed="yes" rot="R270">
 <attribute name="NAME" x="147.7935" y="130.6285" size="0.889" layer="25" ratio="11" rot="R270"/>
 <attribute name="VALUE" x="147.9967" y="127.6186" size="0.6096" layer="27" ratio="10" rot="R270"/>
@@
 <wire x1="121.3237" y1="22.7336" x2="126.1074" y2="22.7336" width="0.3048" layer="1"/>
 </signal>
-<signal name="ONLINE-OFFLINE">
+<signal name="SWITCH">
 <contactref element="R6" pad="2"/>
 <contactref element="S1" pad="2"/>
@@
 <wire x1="121.3237" y1="17.6536" x2="126.1074" y2="17.6536" width="0.3048" layer="1"/>
 </signal>
-<signal name="JOIN_WIFI">
+<signal name="MODE">
 <contactref element="BUTTON" pad="P$1"/>
 <contactref element="BUTTON" pad="P$4"/>
