File: 8x8x8 cube/Base Board.sch (EAGLE design)
At the start: 132 parts, among them J1 CONNECTOR-HEADER-2X2P2X2P-2.5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, J10 CONNECTOR-HEADER-2X2P2X2P-2.5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, J11 CONNECTOR-HEADER-2X2P2X2P-2.5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, J12 CONNECTOR-HEADER-2X2P2X2P-2.5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, J13 CONNECTOR-HEADER-2X2P2X2P-2.5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, J14 CONNECTOR-HEADER-2X2P2X2P-2.5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, J15 CONNECTOR-HEADER-2X2P2X2P-2.5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, J16 CONNECTOR-HEADER-2X2P2X2P-2.5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, J17 CONNECTOR-HEADER-2X2P2X2P-2.5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, J18 CONNECTOR-HEADER-2X2P2X2P-2.5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, J19 CONNECTOR-HEADER-2X2P2X2P-2.5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, J2 CONNECTOR-HEADER-2X2P2X2P-2.5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, J20 CONNECTOR-HEADER-2X2P2X2P-2.5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, J21 CONNECTOR-HEADER-2X2P2X2P-2.5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, J22 CONNECTOR-HEADER-2X2P2X2P-2.5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, J23 CONNECTOR-HEADER-2X2P2X2P-2.5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, J24 CONNECTOR-HEADER-2X2P2X2P-2.5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, J25 CONNECTOR-HEADER-2X2P2X2P-2.5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, J26 CONNECTOR-HEADER-2X2P2X2P-2.5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, J27 CONNECTOR-HEADER-2X2P2X2P-2.5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, J28 CONNECTOR-HEADER-2X2P2X2P-2.5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, J29 CONNECTOR-HEADER-2X2P2X2P-2.5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, J3 CONNECTOR-HEADER-2X2P2X2P-2.5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, J30 CONNECTOR-HEADER-2X2P2X2P-2.5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, J31 CONNECTOR-HEADER-2X2P2X2P-2.5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, J32 CONNECTOR-HEADER-2X2P2X2P-2.5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, J33 CONNECTOR-HEADER-2X2P2X2P-2.5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, J34 CONNECTOR-HEADER-2X2P2X2P-2.5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, J35 CONNECTOR-HEADER-2X2P2X2P-2.5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, J36 CONNECTOR-HEADER-2X2P2X2P-2.5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, J37 CONNECTOR-HEADER-2X2P2X2P-2.5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, J38 CONNECTOR-HEADER-2X2P2X2P-2.5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, J39 CONNECTOR-HEADER-2X2P2X2P-2.5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, J4 CONNECTOR-HEADER-2X2P2X2P-2.5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, J40 CONNECTOR-HEADER-2X2P2X2P-2.5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, J41 CONNECTOR-HEADER-2X2P2X2P-2.5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, J42 CONNECTOR-HEADER-2X2P2X2P-2.5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, J43 CONNECTOR-HEADER-2X2P2X2P-2.5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, J44 CONNECTOR-HEADER-2X2P2X2P-2.5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, J45 CONNECTOR-HEADER-2X2P2X2P-2.5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, J46 CONNECTOR-HEADER-2X2P2X2P-2.5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, J47 CONNECTOR-HEADER-2X2P2X2P-2.5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, J48 CONNECTOR-HEADER-2X2P2X2P-2.5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, J49 CONNECTOR-HEADER-2X2P2X2P-2.5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, J5 CONNECTOR-HEADER-2X2P2X2P-2.5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, J50 CONNECTOR-HEADER-2X2P2X2P-2.5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, J51 CONNECTOR-HEADER-2X2P2X2P-2.5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, J52 CONNECTOR-HEADER-2X2P2X2P-2.5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, J53 CONNECTOR-HEADER-2X2P2X2P-2.5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, J54 CONNECTOR-HEADER-2X2P2X2P-2.5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, J55 CONNECTOR-HEADER-2X2P2X2P-2.5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, J56 CONNECTOR-HEADER-2X2P2X2P-2.5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, J57 CONNECTOR-HEADER-2X2P2X2P-2.5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, J58 CONNECTOR-HEADER-2X2P2X2P-2.5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, J59 CONNECTOR-HEADER-2X2P2X2P-2.5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, J6 CONNECTOR-HEADER-2X2P2X2P-2.5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, J60 CONNECTOR-HEADER-2X2P2X2P-2.5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, J61 CONNECTOR-HEADER-2X2P2X2P-2.5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, J62 CONNECTOR-HEADER-2X2P2X2P-2.5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, J63 CONNECTOR-HEADER-2X2P2X2P-2.5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, J64 CONNECTOR-HEADER-2X2P2X2P-2.5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, J65 CONNECTOR-HEADER-8P-3460290P1, J66 CONNECTOR-HEADER-8P-3460290P1, J67 CONNECTOR-HEADER-8P-3460290P1, J68 CONNECTOR-HEADER-6P-3460270P1, J7 CONNECTOR-HEADER-2X2P2X2P-2.5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, J8 CONNECTOR-HEADER-2X2P2X2P-2.5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, J9 CONNECTOR-HEADER-2X2P2X2P-2.5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, M1 MICROPHONE, Q1 2N7002, Q2 FDD6637, Q3 2N7002, Q4 SS8550, U1 ADXL335, U3 LMV324IDR-1100030P1

Commit message: renamed a couple lines in the schematic
Connections:
- net MODE renamed JOIN_WIFI
- net SWITCH renamed ONLINE-OFFLINE
Other:
- note added: "online/offline switch"
- moved on the sheet: C4, Q1, R1, R2
Changed lines of the file:
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@@
 <text x="-26.67" y="-73.66" size="1.778" layer="97">User IO</text>
 <text x="-160.02" y="-96.52" size="1.778" layer="97">when S1 is connected, the cube is in 'online' mode</text>
+<text x="-76.2" y="-105.41" size="1.778" layer="97">online/offline switch</text>
 </plain>
 <instances>
@@
 <instance part="JP1" gate="G$1" x="-91.44" y="-53.34" rot="R180"/>
 <instance part="JP2" gate="G$1" x="-45.72" y="-55.88" rot="MR180"/>
-<instance part="R1" gate="R" x="-5.08" y="-60.96" rot="R270"/>
-<instance part="R2" gate="R" x="10.16" y="-60.96" smashed="yes" rot="R270">
-<attribute name="NAME" x="10.16" y="-57.15" size="1.27" layer="95" font="vector" ratio="10" rot="R270"/>
-<attribute name="VALUE" x="10.16" y="-60.96" size="1.27" layer="96" font="vector" ratio="10" rot="R270"/>
-</instance>
-<instance part="SUPPLY68" gate="+5V" x="10.16" y="-52.07"/>
+<instance part="R1" gate="R" x="0" y="-60.96" rot="R270"/>
+<instance part="R2" gate="R" x="15.24" y="-60.96" smashed="yes" rot="R270">
+<attribute name="NAME" x="15.24" y="-57.15" size="1.27" layer="95" font="vector" ratio="10" rot="R270"/>
+<attribute name="VALUE" x="15.24" y="-60.96" size="1.27" layer="96" font="vector" ratio="10" rot="R270"/>
+</instance>
+<instance part="SUPPLY68" gate="+5V" x="15.24" y="-52.07"/>
 <instance part="SUPPLY69" gate="GND" x="-125.73" y="-44.45"/>
 <instance part="SUPPLY70" gate="GND" x="-17.78" y="-52.07"/>
@@
 <instance part="R6" gate="R" x="-68.58" y="-91.44" rot="R270"/>
 <instance part="SUPPLY146" gate="GND" x="-83.82" y="-107.95"/>
-<instance part="C4" gate="C" x="2.54" y="-77.47" rot="R180"/>
+<instance part="C4" gate="C" x="7.62" y="-77.47" rot="R180"/>
 <instance part="R9" gate="R" x="123.19" y="-137.16"/>
 <instance part="C6" gate="C" x="63.5" y="-123.19"/>
@@
 <instance part="+3V1" gate="G$1" x="-5.08" y="13.97"/>
 <instance part="+3V2" gate="G$1" x="6.35" y="20.32"/>
-<instance part="+3V3" gate="G$1" x="-1.27" y="-50.8"/>
+<instance part="+3V3" gate="G$1" x="3.81" y="-50.8"/>
 <instance part="+3V4" gate="G$1" x="-27.94" y="-34.29"/>
 <instance part="R13" gate="R" x="54.61" y="-116.84" rot="R90"/>
@@
 <instance part="SUPPLY7" gate="GND" x="-134.62" y="-64.77"/>
 <instance part="+3V10" gate="G$1" x="-68.58" y="-81.28"/>
-<instance part="Q1" gate="Q" x="2.54" y="-68.58" smashed="yes" rot="R270">
-<attribute name="NAME" x="3.81" y="-71.12" size="1.27" layer="95" ratio="10" rot="R270"/>
-<attribute name="VALUE" x="-1.27" y="-68.58" size="1.27" layer="96" ratio="10" rot="R270" display="name"/>
+<instance part="Q1" gate="Q" x="7.62" y="-68.58" smashed="yes" rot="R270">
+<attribute name="NAME" x="8.89" y="-71.12" size="1.27" layer="95" ratio="10" rot="R270"/>
+<attribute name="VALUE" x="3.81" y="-68.58" size="1.27" layer="96" ratio="10" rot="R270" display="name"/>
 </instance>
 <instance part="U1" gate="G$1" x="264.16" y="-133.35" smashed="yes">
@@
 <pinref part="R2" gate="R" pin="1"/>
 <pinref part="SUPPLY68" gate="+5V" pin="+5V"/>
-<wire x1="10.16" y1="-54.61" x2="10.16" y2="-57.15" width="0.1524" layer="91"/>
+<wire x1="15.24" y1="-54.61" x2="15.24" y2="-57.15" width="0.1524" layer="91"/>
 </segment>
 <segment>
@@
 <segment>
 <pinref part="R2" gate="R" pin="2"/>
-<wire x1="7.62" y1="-68.58" x2="10.16" y2="-68.58" width="0.1524" layer="91"/>
-<wire x1="10.16" y1="-68.58" x2="10.16" y2="-64.77" width="0.1524" layer="91"/>
-<junction x="10.16" y="-68.58"/>
-<wire x1="10.16" y1="-68.58" x2="19.05" y2="-68.58" width="0.1524" layer="91"/>
+<wire x1="12.7" y1="-68.58" x2="15.24" y2="-68.58" width="0.1524" layer="91"/>
+<wire x1="15.24" y1="-68.58" x2="15.24" y2="-64.77" width="0.1524" layer="91"/>
+<junction x="15.24" y="-68.58"/>
+<wire x1="15.24" y1="-68.58" x2="19.05" y2="-68.58" width="0.1524" layer="91"/>
 <label x="19.05" y="-68.58" size="1.778" layer="95" xref="yes"/>
 <pinref part="C4" gate="C" pin="1"/>
-<wire x1="6.35" y1="-77.47" x2="10.16" y2="-77.47" width="0.1524" layer="91"/>
-<wire x1="10.16" y1="-77.47" x2="10.16" y2="-68.58" width="0.1524" layer="91"/>
+<wire x1="11.43" y1="-77.47" x2="15.24" y2="-77.47" width="0.1524" layer="91"/>
+<wire x1="15.24" y1="-77.47" x2="15.24" y2="-68.58" width="0.1524" layer="91"/>
 <pinref part="Q1" gate="Q" pin="D"/>
 </segment>
@@
 <segment>
 <pinref part="R1" gate="R" pin="1"/>
-<wire x1="-5.08" y1="-57.15" x2="-1.27" y2="-57.15" width="0.1524" layer="91"/>
-<wire x1="-1.27" y1="-57.15" x2="2.54" y2="-57.15" width="0.1524" layer="91"/>
-<wire x1="2.54" y1="-57.15" x2="2.54" y2="-63.5" width="0.1524" layer="91"/>
-<junction x="-1.27" y="-57.15"/>
+<wire x1="0" y1="-57.15" x2="3.81" y2="-57.15" width="0.1524" layer="91"/>
+<wire x1="3.81" y1="-57.15" x2="7.62" y2="-57.15" width="0.1524" layer="91"/>
+<wire x1="7.62" y1="-57.15" x2="7.62" y2="-63.5" width="0.1524" layer="91"/>
+<junction x="3.81" y="-57.15"/>
 <pinref part="+3V3" gate="G$1" pin="+3V3"/>
-<wire x1="-1.27" y1="-53.34" x2="-1.27" y2="-57.15" width="0.1524" layer="91"/>
+<wire x1="3.81" y1="-53.34" x2="3.81" y2="-57.15" width="0.1524" layer="91"/>
 <pinref part="Q1" gate="Q" pin="G"/>
 </segment>
@@
 <label x="-27.94" y="-68.58" size="1.778" layer="95"/>
 <pinref part="JP2" gate="G$1" pin="12"/>
-<wire x1="-35.56" y1="-68.58" x2="-5.08" y2="-68.58" width="0.1524" layer="91"/>
+<wire x1="-35.56" y1="-68.58" x2="0" y2="-68.58" width="0.1524" layer="91"/>
 <pinref part="R1" gate="R" pin="2"/>
-<wire x1="-5.08" y1="-68.58" x2="-2.54" y2="-68.58" width="0.1524" layer="91"/>
-<wire x1="-5.08" y1="-64.77" x2="-5.08" y2="-68.58" width="0.1524" layer="91"/>
-<junction x="-5.08" y="-68.58"/>
+<wire x1="0" y1="-68.58" x2="2.54" y2="-68.58" width="0.1524" layer="91"/>
+<wire x1="0" y1="-64.77" x2="0" y2="-68.58" width="0.1524" layer="91"/>
+<junction x="0" y="-68.58"/>
 <pinref part="C4" gate="C" pin="2"/>
-<wire x1="-1.27" y1="-77.47" x2="-5.08" y2="-77.47" width="0.1524" layer="91"/>
-<wire x1="-5.08" y1="-77.47" x2="-5.08" y2="-68.58" width="0.1524" layer="91"/>
+<wire x1="3.81" y1="-77.47" x2="0" y2="-77.47" width="0.1524" layer="91"/>
+<wire x1="0" y1="-77.47" x2="0" y2="-68.58" width="0.1524" layer="91"/>
 <pinref part="Q1" gate="Q" pin="S"/>
 <junction x="-35.56" y="-68.58"/>
@@
 </segment>
 </net>
-<net name="SWITCH" class="0">
+<net name="ONLINE-OFFLINE" class="0">
 <segment>
 <pinref part="R6" gate="R" pin="2"/>
@@
 </segment>
 </net>
-<net name="MODE" class="0">
+<net name="JOIN_WIFI" class="0">
 <segment>
 <pinref part="BUTTON" gate="K" pin="A0"/>

Commit message: updated 8x bom, schematic and layout for the baseboard
Parts:
- R13: value 4.3K -> 4.7K
Connections:
- net JOIN_WIFI renamed MODE
- net ONLINE-OFFLINE renamed SWITCH
Other:
- note removed: "online/offline switch"
- note removed: "when S1 is connected, the cube is in 'online' mode"
- moved on the sheet: C4, Q1, R1, R2
